Commit message: bug fixed for other arm_prefixes

File: robots/fr3_duo/fr3_duo.srdf.xacro (robot description, xacro)
@@ -2,6 +2,7 @@
 <robot xmlns:xacro="http://www.ros.org/wiki/xacro" name="fr3">
   <xacro:include filename="$(find franka_description)/robots/common/franka_arm.srdf.xacro"/>
-  <!-- The ID of the robot model to be used -->
-  <xacro:arg name="robot_type" default="fr3" />
+  <!-- The IDs of the robot models to be used -->
+  <xacro:arg name="robot_types" default="['fr3','fr3']" />
+  <xacro:property name="robot_types_list" value="${$(arg robot_types)}" />
   <!-- Should an end-effector be mounted at the flange?" -->
   <xacro:arg name="hand" default="true" />
@@ -40,7 +41,8 @@
   <xacro:macro name="loop" params="i">
       <xacro:unless value="${i == number_of_robots}">
-          <xacro:property name="robot_prefix" value="${arm_prefixes[i]}_"/>
-          <xacro:property name="full_arm_prefix" value="${robot_prefix}fr3_" />
-          <xacro:franka_arm_srdf robot_type="$(arg robot_type)"
+          <xacro:property name="robot_prefix" value="${arm_prefixes_list[i]}_"/>
+          <xacro:property name="robot_type" value="${robot_types_list[i]}"/>
+          <xacro:property name="full_arm_prefix" value="${robot_prefix}${robot_type}_" />
+          <xacro:franka_arm_srdf robot_type="${robot_type}"
                                  hand="$(arg hand)"
                                  ee_id="$(arg ee_id)"
@@ -63,5 +65,9 @@
   <disable_collisions link1="cover_link" link2="mount_link" reason="Adjacent"/>
   <xacro:macro name="cross_arm_loop" params="left_idx right_idx_start right_idx_end">
-      <disable_collisions link1="left_fr3_link${left_idx}" link2="right_fr3_link${right_idx_start}" reason="Never"/>
+      <xacro:property name="robot_prefix_left" value="${arm_prefixes_list[0]}_"/>
+      <xacro:property name="robot_prefix_right" value="${arm_prefixes_list[1]}_"/>
+      <xacro:property name="robot_type_left" value="${robot_types_list[0]}"/>
+      <xacro:property name="robot_type_right" value="${robot_types_list[1]}"/>
+      <disable_collisions link1="${robot_prefix_left}${robot_type_left}_link${left_idx}" link2="${robot_prefix_right}${robot_type_right}_link${right_idx_start}" reason="Never"/>
             <xacro:if value="${right_idx_start &lt; right_idx_end}">
                 <xacro:cross_arm_loop left_idx="${left_idx}" right_idx_start="${right_idx_start + 1}" right_idx_end="${right_idx_end}"/>

Commit message: fix: Adapted the fr3_duo srdf to match the new URDF structure

File: robots/fr3_duo/fr3_duo.srdf.xacro (robot description, xacro)
@@ -39,4 +39,11 @@
       </xacro:if>
   </xacro:macro>
+  <xacro:macro name="disable_mount_collisions" params="full_arm_prefix link2">
+      <disable_collisions link1="${full_arm_prefix}link0" link2="${link2}" reason="Adjacent"/>
+      <disable_collisions link1="${full_arm_prefix}link1" link2="${link2}" reason="Never"/>
+      <disable_collisions link1="${full_arm_prefix}link2" link2="${link2}" reason="Never"/>
+      <disable_collisions link1="${full_arm_prefix}link3" link2="${link2}" reason="Never"/>
+      <disable_collisions link1="${full_arm_prefix}link4" link2="${link2}" reason="Never"/>
+  </xacro:macro>
   <xacro:macro name="loop" params="i">
       <xacro:unless value="${i == number_of_robots}">
@@ -50,18 +57,16 @@
                                  no_prefix='false'/>
           <xacro:missing_self_arm_collisions full_arm_prefix="${full_arm_prefix}"/>
-          <disable_collisions link1="${full_arm_prefix}link0" link2="cover_link" reason="Never"/>
-          <disable_collisions link1="${full_arm_prefix}link1" link2="cover_link" reason="Default"/>
-          <disable_collisions link1="${full_arm_prefix}link2" link2="cover_link" reason="Never"/>
-          <disable_collisions link1="${full_arm_prefix}link3" link2="cover_link" reason="Never"/>
-          <disable_collisions link1="${full_arm_prefix}link0" link2="mount_link" reason="Adjacent"/>
-          <disable_collisions link1="${full_arm_prefix}link1" link2="mount_link" reason="Never"/>
-          <disable_collisions link1="${full_arm_prefix}link2" link2="mount_link" reason="Never"/>
-          <disable_collisions link1="${full_arm_prefix}link3" link2="mount_link" reason="Never"/>
-          <disable_collisions link1="${full_arm_prefix}link4" link2="mount_link" reason="Never"/>
+          <xacro:disable_mount_collisions full_arm_prefix="${full_arm_prefix}" link2="fr3_duo_mount_mounting_point"/>
+          <xacro:disable_mount_collisions full_arm_prefix="${full_arm_prefix}" link2="fr3_duo_mount_origin"/>
+          <xacro:disable_mount_collisions full_arm_prefix="${full_arm_prefix}" link2="fr3_duo_mount_${arm_prefixes_list[i]}"/>
           <xacro:loop i="${i+1}" />
       </xacro:unless>
   </xacro:macro>
   <xacro:loop i="0"/>
-  <disable_collisions link1="cover_link" link2="mount_link" reason="Adjacent"/>
+  <disable_collisions link1="fr3_duo_mount_mounting_point" link2="fr3_duo_mount_origin" reason="Adjacent"/>
+  <disable_collisions link1="fr3_duo_mount_mounting_point" link2="fr3_duo_mount_${arm_prefixes_list[0]}" reason="Adjacent"/>
+  <disable_collisions link1="fr3_duo_mount_mounting_point" link2="fr3_duo_mount_${arm_prefixes_list[1]}" reason="Adjacent"/>
+  <disable_collisions link1="fr3_duo_mount_origin" link2="fr3_duo_mount_${arm_prefixes_list[0]}" reason="Adjacent"/>
+  <disable_collisions link1="fr3_duo_mount_origin" link2="fr3_duo_mount_${arm_prefixes_list[1]}" reason="Adjacent"/>
   <xacro:macro name="cross_arm_loop" params="left_idx right_idx_start right_idx_end">
       <xacro:property name="robot_prefix_left" value="${arm_prefixes_list[0]}_"/>
