Commit message: feat: ros2 control file added for fr3 duo

File: robots/fr3_duo/fr3_duo.xacro (robot description, xacro)
@@ -3,4 +3,6 @@
   <xacro:include filename="$(find franka_description)/robots/common/franka_robot.xacro"/>
   <xacro:include filename="$(find franka_description)/accessories/fr3_duo_mount_v0_3/fr3_duo_mount.xacro"/>
+  <xacro:include filename="$(find franka_description)/accessories/franka_head_v0_2/franka_head.xacro"/>
+  <xacro:include filename="$(find franka_description)/robots/fr3_duo/fr3_duo.ros2_control.xacro"/>
   <xacro:macro
     name="fr3_duo"
@@ -28,8 +30,16 @@
             no_prefix:=false
             is_async:=false
-            thread_priority:=50">
+            thread_priority:=50
+            is_mobile_fr3_duo:=false">
     <xacro:property name="robot_types_list" value="${robot_types}"/>
     <xacro:property name="robot_ips_list" value="${robot_ips}"/>
     <xacro:property name="arm_prefixes_list" value="${arm_prefixes}"/>
+    <!-- For Gazebo: disable ros2_control on individual robots, use unified control instead -->
+    <xacro:if value="${gazebo}">
+      <xacro:property name="ros_control_flag_for_real_hardware" value="false"/>
+    </xacro:if>
+    <xacro:unless value="${gazebo}">
+      <xacro:property name="ros_control_flag_for_real_hardware" value="${ros2_control}"/>
+    </xacro:unless>
     <xacro:mount
       name="mount"
@@ -38,4 +48,5 @@
       right_prefix="${arm_prefixes_list[1]}">
     </xacro:mount>
+    <xacro:head parent="fr3_duo_mount_mounting_point"/>
     <xacro:property name="number_of_robots" value="2"/>
     <xacro:macro name="fr3_duo_loop" params="i">
@@ -62,5 +73,5 @@
           safety_distance="${safety_distance}"
           with_sc="${with_sc}"
-          ros2_control="${ros2_control}"
+          ros2_control="${ros_control_flag_for_real_hardware}"
           robot_ip="${robot_ips_list[i]}"
           use_fake_hardware="${use_fake_hardware}"
@@ -78,4 +89,18 @@
     </xacro:macro>
     <xacro:fr3_duo_loop i="0"/>
+    <!-- Unified ros2_control for both arms -->
+    <xacro:if value="${gazebo and not is_mobile_fr3_duo}">
+      <xacro:fr3_duo_ros2_control
+        robot_types="${robot_types}"
+        arm_prefixes="${arm_prefixes}"
+        robot_ips="${robot_ips}"
+        use_fake_hardware="${use_fake_hardware}"
+        fake_sensor_commands="${fake_sensor_commands}"
+        is_async="${is_async}"
+        thread_priority="${thread_priority}"
+        hand="${hand}"
+        gazebo="${gazebo}"
+        gazebo_effort="${gazebo_effort}"/>
+    </xacro:if>
   </xacro:macro>
 </robot>

File: robots/mobile_fr3_duo_v0_2/mobile_fr3_duo_v0_2.xacro (robot description, xacro)
@@ -26,5 +26,4 @@
             is_async:=false
             thread_priority:=50">
-    <xacro:include filename="$(find franka_description)/accessories/franka_head_v0_2/franka_head.xacro"/>
     <xacro:include filename="$(find franka_description)/accessories/franka_spine_v0_1/franka_spine.xacro"/>
     <xacro:include filename="$(find franka_description)/robots/common/franka_robot.xacro"/>
@@ -63,7 +62,6 @@
       is_async="${is_async}"
       thread_priority="${thread_priority}"/>
-    <!-- Head and Spine -->
+    <!-- Spine -->
     <xacro:franka_spine parent="base_link"/>
-    <xacro:head parent="fr3_duo_mount_mounting_point"/>
     <!-- The FR3 Duo Arms -->
     <xacro:property name="only_arm_robot_types_list" value="${robot_types_list[1:]}"/>
@@ -92,5 +90,6 @@
       arm_prefixes="${arm_prefixes_list}"
       is_async="${is_async}"
-      thread_priority="${thread_priority}"/>
+      thread_priority="${thread_priority}"
+      is_mobile_fr3_duo="true"/>
     <xacro:if value="${gazebo}">
       <xacro:mobile_fr3_duo_ros2_control
