Commit message: feat: adaptations for gazebo

File: robots/common/franka_arm.ros2_control.xacro (robot description, xacro)
@@ -28,5 +28,5 @@
           </xacro:if>
           <xacro:if value="${gazebo}">
-            <plugin>franka_gz_ros2_control/GZSystem</plugin>
+            <plugin>gz_ros2_control/GazeboSimSystem</plugin>
           </xacro:if>
           <xacro:if value="${use_fake_hardware == 0 and gazebo == 0}">
@@ -94,5 +94,5 @@
     <xacro:if value="${gazebo}">
       <gazebo>
-        <plugin filename="franka_gz_ros2_control-system" name="gz_ros2_control::GZROS2ControlPlugin">
+        <plugin filename="gz_ros2_control-system" name="gz_ros2_control::GazeboSimROS2ControlPlugin">
           <parameters>$(find franka_gazebo_bringup)/config/franka_gazebo_controllers.yaml</parameters>
         </plugin>

File: robots/common/franka_arm.xacro (robot description, xacro)
@@ -12,5 +12,5 @@
     <xacro:property name="prefix" value="${'' if no_prefix else arm_prefix + robot_type + '_'}" />
     <xacro:property name="with_accelerometers" value="${'false' if accelerometer_config == 'none' else 'true'}" />
-    <xacro:if value="${gazebo}">
+    <xacro:if value="${gazebo and connected_to == 'base'}">
       <xacro:property name="connected_to" value="" />
     </xacro:if>

File: robots/common/franka_robot.xacro (robot description, xacro)
@@ -98,15 +98,4 @@
     <!-- Definition of additional Gazebo tags -->
     <xacro:if value="${gazebo}">
-      <xacro:if value="${parent != ''}">
-        <!-- Gazebo requires a joint to a link called "world" for statically mounted robots -->
-        <xacro:if value="${parent == 'world'}">
-          <link name="${parent}" />
-        </xacro:if>
-        <joint name="${parent}_joint" type="fixed">
-          <origin xyz="${xyz}" rpy="${rpy}" />
-          <parent link="${parent}" />
-          <child  link="${arm_prefix}${robot_type}_link0" />
-        </joint>
-      </xacro:if>
       <xacro:gazebo-joint joint="${arm_prefix}${robot_type}_joint1" transmission="hardware_interface/PositionJointInterface" />
       <xacro:gazebo-joint joint="${arm_prefix}${robot_type}_joint2" transmission="hardware_interface/PositionJointInterface" />

File: robots/fer/fer.urdf.xacro (robot description, xacro)
@@ -44,4 +44,16 @@
   <xacro:property name="prefix" value="$(arg arm_prefix)"/>
   <xacro:property name="modified_prefix" value="${prefix + '_' if prefix else ''}"/>
+  <!--Position offset with respect the world-->
+  <xacro:arg name="xyz" default="0 0 0" />
+  <!--Rotation offset with respect the world-->
+  <xacro:arg name="rpy" default="0 0 0" />
+  <xacro:if value="$(arg gazebo)">
+    <link name="world" />
+    <joint name="world_joint" type="fixed">
+      <origin xyz="$(arg xyz)" rpy="$(arg rpy)" />
+      <parent link="world" />
+      <child  link="${modified_prefix}$(arg robot_type)_link0" />
+    </joint>
+  </xacro:if>
   <xacro:franka_robot robot_type="fer"
                       joint_limits="${xacro.load_yaml('$(find franka_description)/robots/fer/joint_limits.yaml')}"

File: robots/fp3/fp3.urdf.xacro (robot description, xacro)
@@ -44,4 +44,16 @@
   <xacro:property name="prefix" value="$(arg arm_prefix)"/>
   <xacro:property name="modified_prefix" value="${prefix + '_' if prefix else ''}"/>
+  <!--Position offset with respect the world-->
+  <xacro:arg name="xyz" default="0 0 0" />
+  <!--Rotation offset with respect the world-->
+  <xacro:arg name="rpy" default="0 0 0" />
+  <xacro:if value="$(arg gazebo)">
+    <link name="world" />
+    <joint name="world_joint" type="fixed">
+      <origin xyz="$(arg xyz)" rpy="$(arg rpy)" />
+      <parent link="world" />
+      <child  link="${modified_prefix}$(arg robot_type)_link0" />
+    </joint>
+  </xacro:if>
   <xacro:franka_robot robot_type="fp3"
                       joint_limits="${xacro.load_yaml('$(find franka_description)/robots/fp3/joint_limits.yaml')}"

File: robots/fr3/fr3.urdf.xacro (robot description, xacro)
@@ -44,4 +44,16 @@
   <xacro:property name="prefix" value="$(arg arm_prefix)"/>
   <xacro:property name="modified_prefix" value="${prefix + '_' if prefix else ''}"/>
+  <!--Position offset with respect the world-->
+  <xacro:arg name="xyz" default="0 0 0" />
+  <!--Rotation offset with respect the world-->
+  <xacro:arg name="rpy" default="0 0 0" />
+  <xacro:if value="$(arg gazebo)">
+    <link name="world" />
+    <joint name="world_joint" type="fixed">
+      <origin xyz="$(arg xyz)" rpy="$(arg rpy)" />
+      <parent link="world" />
+      <child  link="${modified_prefix}$(arg robot_type)_link0" />
+    </joint>
+  </xacro:if>
   <xacro:franka_robot robot_type="fr3"
                       joint_limits="${xacro.load_yaml('$(find franka_description)/robots/fr3/joint_limits.yaml')}"

File: robots/fr3_duo/fr3_duo.urdf.xacro (robot description, xacro)
@@ -49,4 +49,16 @@
   <xacro:arg name="arm_prefixes" default="['left','right']" />
   <xacro:property name="arm_prefixes_list" value="${$(arg arm_prefixes)}" />
+  <!--Position offset with respect the world-->
+  <xacro:arg name="xyz" default="0 0 0" />
+  <!--Rotation offset with respect the world-->
+  <xacro:arg name="rpy" default="0 0 0" />
+  <xacro:if value="$(arg gazebo)">
+    <link name="world" />
+    <joint name="world_joint" type="fixed">
+      <origin xyz="$(arg xyz)" rpy="$(arg rpy)" />
+      <parent link="world" />
+      <child  link="${modified_prefix}$(arg robot_type)_link0" />
+    </joint>
+  </xacro:if>
   <link name="base">
   </link>

File: robots/fr3v2/fr3v2.urdf.xacro (robot description, xacro)
@@ -44,4 +44,16 @@
   <xacro:property name="prefix" value="$(arg arm_prefix)"/>
   <xacro:property name="modified_prefix" value="${prefix + '_' if prefix else ''}"/>
+  <!--Position offset with respect the world-->
+  <xacro:arg name="xyz" default="0 0 0" />
+  <!--Rotation offset with respect the world-->
+  <xacro:arg name="rpy" default="0 0 0" />
+  <xacro:if value="$(arg gazebo)">
+    <link name="world" />
+    <joint name="world_joint" type="fixed">
+      <origin xyz="$(arg xyz)" rpy="$(arg rpy)" />
+      <parent link="world" />
+      <child  link="${modified_prefix}$(arg robot_type)_link0" />
+    </joint>
+  </xacro:if>
   <xacro:franka_robot robot_type="fr3v2"
                       joint_limits="${xacro.load_yaml('$(find franka_description)/robots/fr3v2/joint_limits.yaml')}"

File: robots/fr3v2_1/fr3v2_1.urdf.xacro (robot description, xacro)
@@ -44,4 +44,16 @@
   <xacro:property name="prefix" value="$(arg arm_prefix)"/>
   <xacro:property name="modified_prefix" value="${prefix + '_' if prefix else ''}"/>
+  <!--Position offset with respect the world-->
+  <xacro:arg name="xyz" default="0 0 0" />
+  <!--Rotation offset with respect the world-->
+  <xacro:arg name="rpy" default="0 0 0" />
+  <xacro:if value="$(arg gazebo)">
+    <link name="world" />
+    <joint name="world_joint" type="fixed">
+      <origin xyz="$(arg xyz)" rpy="$(arg rpy)" />
+      <parent link="world" />
+      <child  link="${modified_prefix}$(arg robot_type)_link0" />
+    </joint>
+  </xacro:if>
   <xacro:franka_robot robot_type="fr3v2_1"
                       joint_limits="${xacro.load_yaml('$(find franka_description)/robots/fr3v2_1/joint_limits.yaml')}"

File: robots/mobile_fr3_duo_v0_2/mobile_fr3_duo_v0_2.urdf.xacro (robot description, xacro)
@@ -4,4 +4,5 @@
   <xacro:include filename="$(find franka_description)/robots/fr3_duo/fr3_duo_mount/fr3_duo_mount.xacro" />
   <xacro:include filename="$(find franka_description)/robots/tmrv0_2/tmrv0_2.xacro"/>
+  <xacro:include filename="$(find franka_description)/robots/mobile_fr3_duo_v0_2/mobile_fr3_duo.ros2_control.xacro"/>
   <!-- Define arguments -->
   <!-- The IDs of the robot models to be used -->
@@ -43,12 +44,18 @@
   <!-- Name of the description package -->
   <xacro:arg name="description_pkg" default="franka_description" />
-  <!-- Are the robots using the async hardware interface? -->
-  <xacro:arg name="is_async" default="false" />
-  <!-- Thread priority for the hardware interface -->
-  <xacro:arg name="thread_priority" default="50" />
+  <!-- The name of the frame to which the robot is connected. -->
+  <xacro:arg name="connected_to" default="base" />
   <!-- Should the reduced tmr kinematic version (without caster wheels) be used? -->
   <xacro:arg name="reduced_version" default="false" />
-  <link name="base">
-  </link>
+  <!-- Should the arms be used? -->
+  <xacro:arg name="use_arms" default="true" />
+  <xacro:unless value="$(arg gazebo)">
+    <link name="base"/>
+    <joint name="base_joint" type="fixed">
+      <parent link="${fixed_link_name}"/>
+      <child link="base_link"/>
+      <origin rpy="0 0 0" xyz="0 0 0"/>
+    </joint>
+  </xacro:unless>
   <xacro:property name="number_of_robots" value = "3"/>
   <xacro:property name="arm_prefixes_list" value="${['','left','right']}" />
@@ -59,13 +66,9 @@
         <xacro:tmrv0_2 mobile_robot_type="${robot_type_i}"
                 robot_ip="${robot_ips_list[i]}"
-                ros2_control="$(arg ros2_control)"
+                ros2_control="false"
                 use_fake_hardware="$(arg use_fake_hardware)"
                 fake_sensor_commands="$(arg fake_sensor_commands)"
-                reduced_version="$(arg reduced_version)"/>
-        <joint name="base_joint" type="fixed">
-          <parent link="base" />
-          <child link="base_link" />
-          <origin xyz="0 0 0" rpy="0 0 0" />
-        </joint>
+                reduced_version="$(arg reduced_version)"
+                gazebo="$(arg gazebo)"/>
         <link name="franka_spine">
           <visual name="franka_spine_visual">
@@ -99,5 +102,12 @@
           <origin xyz="0.138289 0.0 0.350" rpy="0 0 0" />
         </joint>
-        <link name="franka_spine_support"/>
+        <link name="franka_spine_support">
+          <inertial>
+            <origin xyz="0 0 0" rpy="0 0 0"/>
+            <mass value="0.01"/>
+            <inertia ixx="0.0001" ixy="0.0" ixz="0.0"
+                    iyy="0.0001" iyz="0.0" izz="0.0001"/>
+          </inertial>
+        </link>
         <joint name="franka_spine_vertical_joint" type="prismatic">
           <parent link="franka_spine" />
@@ -113,51 +123,52 @@
       </xacro:if>
       <xacro:unless value="${robot_type_i == 'tmrv0_2'}">
-        <xacro:property name="mount_to_base" value="${xacro.load_yaml('$(arg mount_kinematics)')}"/>
-        <xacro:property name="robot_prefix" value="${arm_prefixes_list[i]}"/>
-        <xacro:property name="modified_prefix" value="${robot_prefix + '_' if robot_prefix else ''}"/>
-        <joint name="${arm_prefixes_list[i]}_base_joint" type="fixed">
-          <parent link="mount_link"/>
-          <child link="${arm_prefixes_list[i]}_base"/>
-          <xacro:if value="${robot_prefix == 'left'}">
-            <xacro:property name="mount_corner" value="${mount_to_base['left']}" lazy_eval="false" />
-          </xacro:if>
-          <xacro:if value="${robot_prefix == 'right'}">
-            <xacro:property name="mount_corner" value="${mount_to_base['right']}" lazy_eval="false" />
-          </xacro:if>
-          <origin rpy="${mount_corner.kinematic.roll} ${mount_corner.kinematic.pitch} ${mount_corner.kinematic.yaw}" xyz="${mount_corner.kinematic.x} ${mount_corner.kinematic.y} ${mount_corner.kinematic.z}"/>
-        </joint>
-        <xacro:arg name="inertials_path" default="$(find franka_description)/robots/${robot_type_i}/inertials.yaml"/>
-        <xacro:arg name="kinematics_path" default="$(find franka_description)/robots/${robot_type_i}/kinematics.yaml"/>
-        <xacro:arg name="dynamics_path" default="$(find franka_description)/robots/${robot_type_i}/dynamics.yaml"/>
-        <xacro:arg name="joint_limits_path" default="$(find franka_description)/robots/${robot_type_i}/joint_limits.yaml"/>
-        <xacro:arg name="accelerometers_path" default="$(find franka_description)/robots/${robot_type_i}/accelerometers.yaml"/>
-        <xacro:franka_robot robot_type="${robot_type_i}"
-                            joint_limits="${xacro.load_yaml('$(arg joint_limits_path)')}"
-                            inertials="${xacro.load_yaml('$(arg inertials_path)')}"
-                            kinematics="${xacro.load_yaml('$(arg kinematics_path)')}"
-                            dynamics="${xacro.load_yaml('$(arg dynamics_path)')}"
-                            accelerometer_config="${xacro.load_yaml('$(arg accelerometers_path)')}"
-                            gazebo="$(arg gazebo)"
-                            hand="$(arg hand)"
-                            ee_id="$(arg ee_id)"
-                            special_connection="$(arg special_connection)"
-                            xyz_ee="$(arg xyz_ee)"
-                            rpy_ee="$(arg rpy_ee)"
-                            tcp_xyz="$(arg tcp_xyz)"
-                            tcp_rpy="$(arg tcp_rpy)"
-                            safety_distance="$(arg safety_distance)"
-                            with_sc="$(arg with_sc)"
-                            ros2_control="$(arg ros2_control)"
-                            robot_ip="${robot_ips_list[i]}"
-                            use_fake_hardware="$(arg use_fake_hardware)"
-                            fake_sensor_commands="$(arg fake_sensor_commands)"
-                            gazebo_effort="$(arg gazebo_effort)"
-                            no_prefix="$(arg no_prefix)"
-                            arm_prefix= "${modified_prefix}"
-                            description_pkg="$(arg description_pkg)"
-                            connected_to="${arm_prefixes_list[i]}_base"
-                            is_async="$(arg is_async)"
-                            thread_priority="$(arg thread_priority)">
-        </xacro:franka_robot>
+        <xacro:if value="$(arg use_arms)">
+          <xacro:property name="mount_to_base" value="${xacro.load_yaml('$(arg mount_kinematics)')}"/>
+          <xacro:property name="robot_prefix" value="${arm_prefixes_list[i]}"/>
+          <xacro:property name="modified_prefix" value="${robot_prefix + '_' if robot_prefix else ''}"/>
+          <joint name="${arm_prefixes_list[i]}_base_joint" type="fixed">
+            <parent link="mount_link"/>
+            <child link="${arm_prefixes_list[i]}_base"/>
+            <xacro:if value="${robot_prefix == 'left'}">
+              <xacro:property name="mount_corner" value="${mount_to_base['left']}" lazy_eval="false" />
+            </xacro:if>
+            <xacro:if value="${robot_prefix == 'right'}">
+              <xacro:property name="mount_corner" value="${mount_to_base['right']}" lazy_eval="false" />
+            </xacro:if>
+            <origin rpy="${mount_corner.kinematic.roll} ${mount_corner.kinematic.pitch} ${mount_corner.kinematic.yaw}" xyz="${mount_corner.kinematic.x} ${mount_corner.kinematic.y} ${mount_corner.kinematic.z}"/>
+          </joint>
+          <xacro:arg name="inertials_path" default="$(find franka_description)/robots/${robot_type_i}/inertials.yaml"/>
+          <xacro:arg name="kinematics_path" default="$(find franka_description)/robots/${robot_type_i}/kinematics.yaml"/>
+          <xacro:arg name="dynamics_path" default="$(find franka_description)/robots/${robot_type_i}/dynamics.yaml"/>
+          <xacro:arg name="joint_limits_path" default="$(find franka_description)/robots/${robot_type_i}/joint_limits.yaml"/>
+          <xacro:arg name="accelerometers_path" default="$(find franka_description)/robots/${robot_type_i}/accelerometers.yaml"/>
+          <xacro:franka_robot robot_type="${robot_type_i}"
+                              joint_limits="${xacro.load_yaml('$(arg joint_limits_path)')}"
+                              inertials="${xacro.load_yaml('$(arg inertials_path)')}"
+                              kinematics="${xacro.load_yaml('$(arg kinematics_path)')}"
+                              dynamics="${xacro.load_yaml('$(arg dynamics_path)')}"
+                              accelerometer_config="${xacro.load_yaml('$(arg accelerometers_path)')}"
+                              gazebo="$(arg gazebo)"
+                              hand="$(arg hand)"
+                              ee_id="$(arg ee_id)"
+                              special_connection="$(arg special_connection)"
+                              xyz_ee="$(arg xyz_ee)"
+                              rpy_ee="$(arg rpy_ee)"
+                              tcp_xyz="$(arg tcp_xyz)"
+                              tcp_rpy="$(arg tcp_rpy)"
+                              safety_distance="$(arg safety_distance)"
+                              with_sc="$(arg with_sc)"
+                              ros2_control="false"
+                              robot_ip="${robot_ips_list[i]}"
+                              use_fake_hardware="$(arg use_fake_hardware)"
+                              fake_sensor_commands="$(arg fake_sensor_commands)"
+                              gazebo_effort="$(arg gazebo_effort)"
+                              no_prefix="$(arg no_prefix)"
+                              arm_prefix= "${modified_prefix}"
+                              description_pkg="$(arg description_pkg)"
+                              connected_to="${arm_prefixes_list[i]}_base"
+                              parent="${arm_prefixes_list[i]}_base">
+          </xacro:franka_robot>
+        </xacro:if>
       </xacro:unless>
       <xacro:loop i="${i+1}"/>
@@ -165,3 +176,12 @@
   </xacro:macro>
   <xacro:loop i="0"/>
+  <xacro:mobile_fr3_duo_ros2_control mobile_robot_type="tmrv0_2"
+                                     robot_types="${robot_types_list}"
+                                     arm_prefixes="${arm_prefixes_list}"
+                                     robot_ips="${robot_ips_list}"
+                                     use_fake_hardware="$(arg use_fake_hardware)"
+                                     fake_sensor_commands="$(arg fake_sensor_commands)"
+                                     gazebo="$(arg gazebo)"
+                                     gazebo_effort="$(arg gazebo_effort)"
+                                     robot_namespace=""/>
 </robot>

File: robots/tmrv0_2/argo_drive.xacro (robot description, xacro)
@@ -7,5 +7,5 @@
     <xacro:property name="base_height" value="0.077" />
     <xacro:property name="offset_wheel" value="0.085" />
-    <xacro:property name="mass" value="0.5" />
+    <xacro:property name="mass" value="2.5" />
     <xacro:if value="${name == 'argo_drive_front'}">
       <xacro:property name="steering_joint" value="0" />
@@ -49,5 +49,13 @@
       <child  link="${name}_fixed_link" />
     </joint>
-    <link name="${name}_steering_link" />
+    <link name="${name}_steering_link">
+     <inertial>
+        <origin xyz="0 0 0" rpy="0 0 0"/>
+        <mass value="2.0"/>
+        <inertia ixx="0.1" ixy="0.0" ixz="0.0"
+                 iyy="0.1" iyz="0.0"
+                 izz="0.1"/>
+      </inertial>
+    </link>
     <joint name="${mobile_robot_type}_joint_${steering_joint}" type="continuous">
       <origin xyz="0 0 0"/>
@@ -56,5 +64,5 @@
       <axis   xyz="0 0 1" />
       <limit  effort="500" velocity="20" />
-      <dynamics damping="0.003" friction="0.0"/>
+      <dynamics damping="20.0" friction="5.0"/>
     </joint>
     <link name="${name}_link" >
@@ -81,6 +89,6 @@
       <child  link="${name}_link" />
       <axis   xyz="0 1 0" />
-      <limit  effort="500" velocity="20" />
-      <dynamics damping="0.003" friction="0.0"/>
+      <limit  effort="500" velocity="20"/>
+      <dynamics damping="5.0" friction="1.0"/>
     </joint>
   </xacro:macro>

File: robots/tmrv0_2/caster_wheel.xacro (robot description, xacro)
@@ -40,5 +40,13 @@
       <child  link="${name}_fixed_link" />
     </joint>
-    <link name="${name}_steering_link" />
+    <link name="${name}_steering_link">
+      <inertial>
+          <origin xyz="0 0 0" rpy="0 0 0"/>
+          <mass value="0.01"/>
+          <inertia ixx="0.0001" ixy="0.0" ixz="0.0"
+                   iyy="0.0001" iyz="0.0"
+                   izz="0.0001"/>
+      </inertial>
+    </link>
     <joint name="${name}_steering_joint" type="continuous">
       <origin xyz="0 0 0"/>
@@ -65,4 +73,11 @@
         <xacro:caster_wheel_geometry/>
       </collision>
+      <inertial>
+        <origin xyz="0 0 0" rpy="0 0 0"/>
+        <mass value="0.001"/>
+        <inertia ixx="0.0001" ixy="0.0" ixz="0.0"
+                 iyy="0.0001" iyz="0.0"
+                 izz="0.0001"/>
+      </inertial>
     </link>
     <joint name="${name}_joint" type="continuous">
