Commit message: feat: adaptations for gazebo

File: robots/tmrv0_2/tmrv0_2.ros2_control.xacro (robot description, xacro)
@@ -7,5 +7,7 @@
             fake_sensor_commands
             is_async:=false
-            thread_priority:=50">
+            thread_priority:=50
+            gazebo
+            robot_namespace">
     <ros2_control name="TmrHardware" type="system" is_async="${is_async}">
       <xacro:if value="${is_async}">
@@ -23,5 +25,11 @@
           <param name="state_following_offset">0.0</param>
         </xacro:if>
-        <xacro:if value="${use_fake_hardware == 0}">
+        <xacro:if value="${gazebo}">
+          <plugin>gz_ros2_control/GazeboSimSystem</plugin>
+          <plugin>fake_components/GenericSystem</plugin>
+          <param name="fake_sensor_commands">${fake_sensor_commands}</param>
+          <param name="state_following_offset">0.0</param>
+        </xacro:if>
+        <xacro:if value="${use_fake_hardware == 0 and gazebo == 0}">
           <plugin>franka_hardware/FrankaHardwareInterface</plugin>
           <param name="robot_ip">${robot_ip}</param>
@@ -34,4 +42,7 @@
             <param name="initial_value">0.0</param>
           </state_interface>
+          <state_interface name="velocity">
+            <param name="initial_value">0.0</param>
+          </state_interface>
         </joint>
       </xacro:macro>
@@ -39,4 +50,7 @@
         <joint name="${joint_name}">
           <command_interface name="velocity"/>
+          <state_interface name="position">
+            <param name="initial_value">0.0</param>
+          </state_interface>
           <state_interface name="velocity">
             <param name="initial_value">0.0</param>
@@ -48,4 +62,49 @@
       <xacro:configure_steering_joint joint_name="${mobile_robot_type}_joint_2"/>
       <xacro:configure_driving_joint joint_name="${mobile_robot_type}_joint_3"/>
+       <!-- Rocker Arm -->
+      <joint name="rocker_arm_joint">
+        <state_interface name="position">
+          <param name="initial_value">0.0</param>
+        </state_interface>
+        <state_interface name="velocity">
+          <param name="initial_value">0.0</param>
+        </state_interface>
+      </joint>
+      <!-- Front caster steering -->
+      <joint name="caster_front_left_steering_joint">
+        <state_interface name="position">
+          <param name="initial_value">0.0</param>
+        </state_interface>
+        <state_interface name="velocity">
+          <param name="initial_value">0.0</param>
+        </state_interface>
+      </joint>
+      <!-- Front caster joint -->
+      <joint name="caster_front_left_joint">
+        <state_interface name="position">
+          <param name="initial_value">0.0</param>
+        </state_interface>
+        <state_interface name="velocity">
+          <param name="initial_value">0.0</param>
+        </state_interface>
+      </joint>
+      <!-- Rear caster steering -->
+      <joint name="caster_rear_right_steering_joint">
+        <state_interface name="position">
+          <param name="initial_value">0.0</param>
+        </state_interface>
+        <state_interface name="velocity">
+          <param name="initial_value">0.0</param>
+        </state_interface>
+      </joint>
+      <!-- Rear caster joint -->
+      <joint name="caster_rear_right_joint">
+        <state_interface name="position">
+          <param name="initial_value">0.0</param>
+        </state_interface>
+        <state_interface name="velocity">
+          <param name="initial_value">0.0</param>
+        </state_interface>
+      </joint>
       <xacro:macro name="general_purpose_io" params="prefix command_interface index">
         <gpio name="${prefix}">
@@ -62,4 +121,11 @@
       <xacro:general_purpose_io prefix="wz" command_interface="cartesian_velocity" index="5"/>
     </ros2_control>
+    <xacro:if value="${gazebo}">
+      <gazebo>
+        <plugin filename="gz_ros2_control-system" name="gz_ros2_control::GazeboSimROS2ControlPlugin">
+          <parameters>$(find franka_gazebo_bringup)/config/franka_gazebo_controllers.yaml</parameters>
+        </plugin>
+      </gazebo>
+    </xacro:if>y
   </xacro:macro>
 </robot>

File: robots/tmrv0_2/tmrv0_2.urdf.xacro (robot description, xacro)
@@ -15,11 +15,16 @@
   <!-- Should the reduced kinematic version (without caster wheels) be used? -->
   <xacro:arg name="reduced_version" default="false" />
-  <link name="base">
-  </link>
-  <joint name="base_joint" type="fixed">
-    <parent link="base"/>
-    <child link="base_link"/>
-    <origin rpy="0 0 0" xyz="0 0 0"/>
-  </joint>
+  <!-- Should the robot be spawned in Gazebo?" -->
+  <xacro:arg name="gazebo" default="false" />
+  <!-- The namespace of the robot -->
+  <xacro:arg name="robot_namespace" default="" />
+  <xacro:unless value="$(arg gazebo)">
+    <link name="base"/>
+    <joint name="base_joint" type="fixed">
+      <parent link="base"/>
+      <child link="base_link"/>
+      <origin rpy="0 0 0" xyz="0 0 0"/>
+    </joint>
+  </xacro:unless>
   <xacro:tmrv0_2 mobile_robot_type="$(arg robot_type)"
               robot_ip="$(arg robot_ip)"
@@ -27,4 +32,6 @@
               use_fake_hardware="$(arg use_fake_hardware)"
               fake_sensor_commands="$(arg fake_sensor_commands)"
-              reduced_version="$(arg reduced_version)"/>
+              reduced_version="$(arg reduced_version)"
+              robot_namespace="$(arg robot_namespace)"
+              gazebo="$(arg gazebo)"/>
 </robot>

File: robots/tmrv0_2/tmrv0_2.xacro (robot description, xacro)
@@ -9,5 +9,7 @@
                   reduced_version:=false
                   is_async:=false
-                  thread_priority:=50">
+                  thread_priority:=50
+                  robot_namespace:=''
+                  gazebo:=false">
     <xacro:include filename="$(find franka_description)/robots/tmrv0_2/argo_drive.xacro" />
     <xacro:include filename="$(find franka_description)/robots/tmrv0_2/caster_wheel.xacro" />
@@ -141,4 +143,6 @@
         use_fake_hardware="${use_fake_hardware}"
         fake_sensor_commands="${fake_sensor_commands}"
+        robot_namespace="${robot_namespace}"
+        gazebo="${gazebo}"
       />
     </xacro:if>
