Commit message: refactor: Moving ros2_control related parts to franka_ros2

File: robots/common/franka_robot.xacro (robot description, xacro)
@@ -16,15 +16,8 @@
                       gazebo:='false'
                       with_sc:='false'
-                      ros2_control:=false
-                      robot_ip:=''
-                      use_fake_hardware:=false
-                      fake_sensor_commands:=false
-                      gazebo_effort:=false
                       no_prefix:='false'
                       arm_prefix:=''
                       description_pkg:='franka_description'
-                      connected_to:='base'
-                      is_async:=false
-                      thread_priority:=50">
+                      connected_to:='base'">
     <xacro:include filename="$(find franka_description)/robots/common/utils.xacro"/>
     <xacro:include filename="$(find franka_description)/robots/common/franka_arm.xacro"/>
@@ -148,19 +141,4 @@
       </xacro:if>
     </xacro:if>
-    <xacro:if value="${ros2_control}">
-      <xacro:include filename="$(find franka_description)/robots/common/franka_arm.ros2_control.xacro"/>
-      <xacro:franka_arm_ros2_control
-        robot_type="${robot_type}"
-        robot_ip="${robot_ip}"
-        use_fake_hardware="${use_fake_hardware}"
-        fake_sensor_commands="${fake_sensor_commands}"
-        gazebo="${gazebo}"
-        hand="${hand}"
-        gazebo_effort="${gazebo_effort}"
-        arm_prefix="${arm_prefix}"
-        is_async="${is_async}"
-        thread_priority="${thread_priority}"
-      />
-    </xacro:if>
   </xacro:macro>
 </robot>

File: robots/fer/fer.urdf.xacro (robot description, xacro)
@@ -27,16 +27,6 @@
   <!-- Should self-collision be enabled? -->
   <xacro:arg name="with_sc" default="false"/>
-  <!-- Is the robot being controlled with ros2_control?" -->
-  <xacro:arg name="ros2_control" default="false"/>
-  <!-- IP address or hostname of the robot" -->
-  <xacro:arg name="robot_ip" default=""/>
-  <!-- Should a fake hardware be used? -->
-  <xacro:arg name="use_fake_hardware" default="false"/>
-  <!-- Should fake sensors be used? -->
-  <xacro:arg name="fake_sensor_commands" default="false"/>
   <!-- Should the robot be spawned in Gazebo?" -->
   <xacro:arg name="gazebo" default="false"/>
-  <!-- Should the robot be spawned in Gazebo with effort interfaces?" -->
-  <xacro:arg name="gazebo_effort" default="false"/>
   <!-- Name of the description package -->
   <xacro:arg name="description_pkg" default="franka_description"/>
@@ -69,9 +59,4 @@
     safety_distance="$(arg safety_distance)"
     with_sc="$(arg with_sc)"
-    ros2_control="$(arg ros2_control)"
-    robot_ip="$(arg robot_ip)"
-    use_fake_hardware="$(arg use_fake_hardware)"
-    fake_sensor_commands="$(arg fake_sensor_commands)"
-    gazebo_effort="$(arg gazebo_effort)"
     no_prefix="$(arg no_prefix)"
     arm_prefix="${modified_prefix}"

File: robots/fp3/fp3.urdf.xacro (robot description, xacro)
@@ -27,16 +27,6 @@
   <!-- Should self-collision be enabled? -->
   <xacro:arg name="with_sc" default="false"/>
-  <!-- Is the robot being controlled with ros2_control?" -->
-  <xacro:arg name="ros2_control" default="false"/>
-  <!-- IP address or hostname of the robot" -->
-  <xacro:arg name="robot_ip" default=""/>
-  <!-- Should a fake hardware be used? -->
-  <xacro:arg name="use_fake_hardware" default="false"/>
-  <!-- Should fake sensors be used? -->
-  <xacro:arg name="fake_sensor_commands" default="false"/>
   <!-- Should the robot be spawned in Gazebo?" -->
   <xacro:arg name="gazebo" default="false"/>
-  <!-- Should the robot be spawned in Gazebo with effort interfaces?" -->
-  <xacro:arg name="gazebo_effort" default="false"/>
   <!-- Name of the description package -->
   <xacro:arg name="description_pkg" default="franka_description"/>
@@ -69,9 +59,4 @@
     safety_distance="$(arg safety_distance)"
     with_sc="$(arg with_sc)"
-    ros2_control="$(arg ros2_control)"
-    robot_ip="$(arg robot_ip)"
-    use_fake_hardware="$(arg use_fake_hardware)"
-    fake_sensor_commands="$(arg fake_sensor_commands)"
-    gazebo_effort="$(arg gazebo_effort)"
     no_prefix="$(arg no_prefix)"
     arm_prefix="${modified_prefix}"

File: robots/fr3/fr3.urdf.xacro (robot description, xacro)
@@ -27,16 +27,6 @@
   <!-- Should self-collision be enabled? -->
   <xacro:arg name="with_sc" default="false"/>
-  <!-- Is the robot being controlled with ros2_control?" -->
-  <xacro:arg name="ros2_control" default="false"/>
-  <!-- IP address or hostname of the robot" -->
-  <xacro:arg name="robot_ip" default=""/>
-  <!-- Should a fake hardware be used? -->
-  <xacro:arg name="use_fake_hardware" default="false"/>
-  <!-- Should fake sensors be used? -->
-  <xacro:arg name="fake_sensor_commands" default="false"/>
   <!-- Should the robot be spawned in Gazebo?" -->
   <xacro:arg name="gazebo" default="false"/>
-  <!-- Should the robot be spawned in Gazebo with effort interfaces?" -->
-  <xacro:arg name="gazebo_effort" default="false"/>
   <!-- Name of the description package -->
   <xacro:arg name="description_pkg" default="franka_description"/>
@@ -69,9 +59,4 @@
     safety_distance="$(arg safety_distance)"
     with_sc="$(arg with_sc)"
-    ros2_control="$(arg ros2_control)"
-    robot_ip="$(arg robot_ip)"
-    use_fake_hardware="$(arg use_fake_hardware)"
-    fake_sensor_commands="$(arg fake_sensor_commands)"
-    gazebo_effort="$(arg gazebo_effort)"
     no_prefix="$(arg no_prefix)"
     arm_prefix="${modified_prefix}"

File: robots/fr3_duo/fr3_duo.urdf.xacro (robot description, xacro)
@@ -26,23 +26,8 @@
   <!-- Should self-collision be enabled? -->
   <xacro:arg name="with_sc" default="false"/>
-  <!-- Is the robot being controlled with ros2_control?" -->
-  <xacro:arg name="ros2_control" default="false"/>
-  <!-- IP address or hostname of the robot" -->
-  <xacro:arg name="robot_ips" default="['172.16.0.2','172.16.0.3']"/>
-  <xacro:property name="robot_ips_list" value="${$(arg robot_ips)}"/>
-  <!-- Should a fake hardware be used? -->
-  <xacro:arg name="use_fake_hardware" default="false"/>
-  <!-- Should fake sensors be used? -->
-  <xacro:arg name="fake_sensor_commands" default="false"/>
   <!-- Should the robot be spawned in Gazebo?" -->
   <xacro:arg name="gazebo" default="false"/>
-  <!-- Should the robot be spawned in Gazebo with effort interfaces?" -->
-  <xacro:arg name="gazebo_effort" default="false"/>
   <!-- Name of the description package -->
   <xacro:arg name="description_pkg" default="franka_description"/>
-  <!-- Are the robots using the async hardware interface? -->
-  <xacro:arg name="is_async" default="false"/>
-  <!-- Thread priority for the hardware interface -->
-  <xacro:arg name="thread_priority" default="50"/>
   <!-- Arm prefixes of the robots -->
   <xacro:arg name="arm_prefixes" default="['left','right']"/>
@@ -77,16 +62,9 @@
     safety_distance="$(arg safety_distance)"
     with_sc="$(arg with_sc)"
-    ros2_control="$(arg ros2_control)"
     gazebo="$(arg gazebo)"
-    gazebo_effort="$(arg gazebo_effort)"
-    use_fake_hardware="$(arg use_fake_hardware)"
-    fake_sensor_commands="$(arg fake_sensor_commands)"
-    robot_ips="${robot_ips_list}"
     description_pkg="$(arg description_pkg)"
     base_mount="${base_mount_str}"
     connected_to="${base_mount_str}"
     arm_prefixes="${arm_prefixes_list}"
-    no_prefix="$(arg no_prefix)"
-    is_async="$(arg is_async)"
-    thread_priority="$(arg thread_priority)"/>
+    no_prefix="$(arg no_prefix)"/>
 </robot>

File: robots/fr3_duo/fr3_duo.xacro (robot description, xacro)
@@ -4,5 +4,4 @@
   <xacro:include filename="$(find franka_description)/accessories/fr3_duo_mount_v0_3/fr3_duo_mount.xacro"/>
   <xacro:include filename="$(find franka_description)/accessories/franka_head_v0_2/franka_head.xacro"/>
-  <xacro:include filename="$(find franka_description)/robots/fr3_duo/fr3_duo.ros2_control.xacro"/>
   <xacro:macro
     name="fr3_duo"
@@ -18,10 +17,5 @@
             safety_distance
             with_sc
-            ros2_control
             gazebo
-            gazebo_effort
-            use_fake_hardware
-            fake_sensor_commands
-            robot_ips
             description_pkg
             base_mount
@@ -29,17 +23,7 @@
             arm_prefixes
             no_prefix:=false
-            is_async:=false
-            thread_priority:=50
             is_mobile_fr3_duo:=false">
     <xacro:property name="robot_types_list" value="${robot_types}"/>
-    <xacro:property name="robot_ips_list" value="${robot_ips}"/>
     <xacro:property name="arm_prefixes_list" value="${arm_prefixes}"/>
-    <!-- For Gazebo: disable ros2_control on individual robots, use unified control instead -->
-    <xacro:if value="${gazebo}">
-      <xacro:property name="ros_control_flag_for_real_hardware" value="false"/>
-    </xacro:if>
-    <xacro:unless value="${gazebo}">
-      <xacro:property name="ros_control_flag_for_real_hardware" value="${ros2_control}"/>
-    </xacro:unless>
     <xacro:mount
       name="mount"
@@ -73,15 +57,8 @@
           safety_distance="${safety_distance}"
           with_sc="${with_sc}"
-          ros2_control="${ros_control_flag_for_real_hardware}"
-          robot_ip="${robot_ips_list[i]}"
-          use_fake_hardware="${use_fake_hardware}"
-          fake_sensor_commands="${fake_sensor_commands}"
-          gazebo_effort="${gazebo_effort}"
           no_prefix="${no_prefix}"
           arm_prefix="${modified_prefix}"
           description_pkg="${description_pkg}"
-          connected_to="${arm_prefixes_list[i]}_base"
-          is_async="${is_async}"
-          thread_priority="${thread_priority}">
+          connected_to="${arm_prefixes_list[i]}_base">
         </xacro:franka_robot>
         <xacro:fr3_duo_loop i="${i+1}"/>
@@ -89,18 +66,4 @@
     </xacro:macro>
     <xacro:fr3_duo_loop i="0"/>
-    <!-- Unified ros2_control for both arms -->
-    <xacro:if value="${gazebo and not is_mobile_fr3_duo}">
-      <xacro:fr3_duo_ros2_control
-        robot_types="${robot_types}"
-        arm_prefixes="${arm_prefixes}"
-        robot_ips="${robot_ips}"
-        use_fake_hardware="${use_fake_hardware}"
-        fake_sensor_commands="${fake_sensor_commands}"
-        is_async="${is_async}"
-        thread_priority="${thread_priority}"
-        hand="${hand}"
-        gazebo="${gazebo}"
-        gazebo_effort="${gazebo_effort}"/>
-    </xacro:if>
   </xacro:macro>
 </robot>

File: robots/fr3v2/fr3v2.urdf.xacro (robot description, xacro)
@@ -27,16 +27,6 @@
   <!-- Should self-collision be enabled? -->
   <xacro:arg name="with_sc" default="false"/>
-  <!-- Is the robot being controlled with ros2_control?" -->
-  <xacro:arg name="ros2_control" default="false"/>
-  <!-- IP address or hostname of the robot" -->
-  <xacro:arg name="robot_ip" default=""/>
-  <!-- Should a fake hardware be used? -->
-  <xacro:arg name="use_fake_hardware" default="false"/>
-  <!-- Should fake sensors be used? -->
-  <xacro:arg name="fake_sensor_commands" default="false"/>
   <!-- Should the robot be spawned in Gazebo?" -->
   <xacro:arg name="gazebo" default="false"/>
-  <!-- Should the robot be spawned in Gazebo with effort interfaces?" -->
-  <xacro:arg name="gazebo_effort" default="false"/>
   <!-- Name of the description package -->
   <xacro:arg name="description_pkg" default="franka_description"/>
@@ -69,9 +59,4 @@
     safety_distance="$(arg safety_distance)"
     with_sc="$(arg with_sc)"
-    ros2_control="$(arg ros2_control)"
-    robot_ip="$(arg robot_ip)"
-    use_fake_hardware="$(arg use_fake_hardware)"
-    fake_sensor_commands="$(arg fake_sensor_commands)"
-    gazebo_effort="$(arg gazebo_effort)"
     no_prefix="$(arg no_prefix)"
     arm_prefix="${modified_prefix}"

File: robots/fr3v2_1/fr3v2_1.urdf.xacro (robot description, xacro)
@@ -27,16 +27,6 @@
   <!-- Should self-collision be enabled? -->
   <xacro:arg name="with_sc" default="false"/>
-  <!-- Is the robot being controlled with ros2_control?" -->
-  <xacro:arg name="ros2_control" default="false"/>
-  <!-- IP address or hostname of the robot" -->
-  <xacro:arg name="robot_ip" default=""/>
-  <!-- Should a fake hardware be used? -->
-  <xacro:arg name="use_fake_hardware" default="false"/>
-  <!-- Should fake sensors be used? -->
-  <xacro:arg name="fake_sensor_commands" default="false"/>
   <!-- Should the robot be spawned in Gazebo?" -->
   <xacro:arg name="gazebo" default="false"/>
-  <!-- Should the robot be spawned in Gazebo with effort interfaces?" -->
-  <xacro:arg name="gazebo_effort" default="false"/>
   <!-- Name of the description package -->
   <xacro:arg name="description_pkg" default="franka_description"/>
@@ -69,9 +59,4 @@
     safety_distance="$(arg safety_distance)"
     with_sc="$(arg with_sc)"
-    ros2_control="$(arg ros2_control)"
-    robot_ip="$(arg robot_ip)"
-    use_fake_hardware="$(arg use_fake_hardware)"
-    fake_sensor_commands="$(arg fake_sensor_commands)"
-    gazebo_effort="$(arg gazebo_effort)"
     no_prefix="$(arg no_prefix)"
     arm_prefix="${modified_prefix}"

File: robots/mobile_fr3_duo_v0_2/mobile_fr3_duo_v0_2.srdf.xacro (robot description, xacro)
@@ -332,3 +332,6 @@
     <disable_collisions link1="fr3_duo_mount_mounting_point" link2="left_fr3v2_link0" reason="Adjacent"/>
     <disable_collisions link1="fr3_duo_mount_mounting_point" link2="right_fr3v2_link0" reason="Adjacent"/>
+    <disable_collisions link1="fr3_duo_mount_mounting_point" link2="franka_spine" reason="Never"/>
+    <disable_collisions link1="fr3_duo_mount_mounting_point" link2="left_fr3v2_link1" reason="Never"/>
+    <disable_collisions link1="fr3_duo_mount_mounting_point" link2="right_fr3v2_link1" reason="Never"/>
 `</robot>

File: robots/mobile_fr3_duo_v0_2/mobile_fr3_duo_v0_2.urdf.xacro (robot description, xacro)
@@ -26,23 +26,8 @@
   <!-- Should self-collision be enabled? -->
   <xacro:arg name="with_sc" default="false"/>
-  <!-- Is the robot being controlled with ros2_control?" -->
-  <xacro:arg name="ros2_control" default="false"/>
-  <!-- IP address or hostname of the robot" -->
-  <xacro:arg name="robot_ips" default="['172.16.0.1','172.16.0.2','172.16.0.3']"/>
-  <xacro:property name="robot_ips_list" value="${$(arg robot_ips)}"/>
-  <!-- Should a fake hardware be used? -->
-  <xacro:arg name="use_fake_hardware" default="false"/>
-  <!-- Should fake sensors be used? -->
-  <xacro:arg name="fake_sensor_commands" default="false"/>
   <!-- Should the robot be spawned in Gazebo?" -->
   <xacro:arg name="gazebo" default="false"/>
-  <!-- Should the robot be spawned in Gazebo with effort interfaces?" -->
-  <xacro:arg name="gazebo_effort" default="false"/>
   <!-- Name of the description package -->
   <xacro:arg name="description_pkg" default="franka_description"/>
-  <!-- Are the robots using the async hardware interface? -->
-  <xacro:arg name="is_async" default="false"/>
-  <!-- Thread priority for the hardware interface -->
-  <xacro:arg name="thread_priority" default="50"/>
   <!-- The name of the frame to which the robot is connected. -->
   <xacro:arg name="connected_to" default="base"/>
@@ -54,11 +39,6 @@
     robot_types="$(arg robot_types)"
     hand="$(arg hand)"
-    ros2_control="$(arg ros2_control)"
     gazebo="$(arg gazebo)"
-    gazebo_effort="$(arg gazebo_effort)"
-    use_fake_hardware="$(arg use_fake_hardware)"
-    fake_sensor_commands="$(arg fake_sensor_commands)"
     reduced_version="$(arg reduced_version)"
-    robot_ips="$(arg robot_ips)"
     description_pkg="$(arg description_pkg)"
     connected_to="$(arg connected_to)"
@@ -72,6 +52,4 @@
     tcp_rpy="$(arg tcp_rpy)"
     safety_distance="$(arg safety_distance)"
-    with_sc="$(arg with_sc)"
-    is_async="$(arg is_async)"
-    thread_priority="$(arg thread_priority)"/>
+    with_sc="$(arg with_sc)"/>
 </robot>

File: robots/mobile_fr3_duo_v0_2/mobile_fr3_duo_v0_2.xacro (robot description, xacro)
@@ -5,11 +5,6 @@
     params="robot_types
             hand
-            ros2_control
             gazebo
-            gazebo_effort
-            use_fake_hardware
-            fake_sensor_commands
             reduced_version
-            robot_ips
             description_pkg
             connected_to
@@ -23,18 +18,9 @@
             tcp_rpy
             safety_distance
-            with_sc
-            is_async:=false
-            thread_priority:=50">
+            with_sc">
     <xacro:include filename="$(find franka_description)/accessories/franka_spine_v0_1/franka_spine.xacro"/>
     <xacro:include filename="$(find franka_description)/robots/common/franka_robot.xacro"/>
     <xacro:include filename="$(find franka_description)/robots/tmrv0_2/tmrv0_2.xacro"/>
-    <xacro:include filename="$(find franka_description)/robots/mobile_fr3_duo_v0_2/mobile_fr3_duo.ros2_control.xacro"/>
     <xacro:include filename="$(find franka_description)/robots/fr3_duo/fr3_duo.xacro"/>
-    <xacro:if value="${gazebo}">
-      <xacro:property name="ros_control_flag_for_real_hardware" value="false"/>
-    </xacro:if>
-    <xacro:unless value="${gazebo}">
-      <xacro:property name="ros_control_flag_for_real_hardware" value="${ros2_control}"/>
-    </xacro:unless>
     <xacro:property name="arm_prefixes_list" value="${['left','right']}"/>
     <!-- Verify that the given robot types are first a mobile base and then arms -->
@@ -54,17 +40,10 @@
     <xacro:tmrv0_2
       mobile_robot_type="${robot_types_list[0]}"
-      robot_ip="${robot_ips_list[0]}"
-      ros2_control="${ros_control_flag_for_real_hardware}"
-      use_fake_hardware="${use_fake_hardware}"
-      fake_sensor_commands="${fake_sensor_commands}"
       reduced_version="${reduced_version}"
-      gazebo="${gazebo}"
-      is_async="${is_async}"
-      thread_priority="${thread_priority}"/>
+      gazebo="${gazebo}"/>
     <!-- Spine -->
     <xacro:franka_spine parent="base_link"/>
     <!-- The FR3 Duo Arms -->
     <xacro:property name="only_arm_robot_types_list" value="${robot_types_list[1:]}"/>
-    <xacro:property name="only_arm_robot_ips_list" value="${robot_ips_list[1:]}"/>
     <xacro:fr3_duo
       name="fr3_duo"
@@ -79,30 +58,10 @@
       safety_distance="${safety_distance}"
       with_sc="${with_sc}"
-      ros2_control="${ros_control_flag_for_real_hardware}"
       gazebo="${gazebo}"
-      gazebo_effort="${gazebo_effort}"
-      use_fake_hardware="${use_fake_hardware}"
-      fake_sensor_commands="${fake_sensor_commands}"
-      robot_ips="${only_arm_robot_ips_list}"
       description_pkg="${description_pkg}"
       base_mount="franka_spine_mounting_point"
       connected_to="${connected_to}"
       arm_prefixes="${arm_prefixes_list}"
-      is_async="${is_async}"
-      thread_priority="${thread_priority}"
       is_mobile_fr3_duo="true"/>
-    <xacro:if value="${gazebo}">
-      <xacro:mobile_fr3_duo_ros2_control
-        mobile_robot_type="tmrv0_2"
-        robot_types="${robot_types_list}"
-        arm_prefixes="${arm_prefixes_list}"
-        robot_ips="${robot_ips_list}"
-        hand="${hand}"
-        use_fake_hardware="${use_fake_hardware}"
-        fake_sensor_commands="${fake_sensor_commands}"
-        gazebo="${gazebo}"
-        gazebo_effort="${gazebo_effort}"
-        robot_namespace=""/>
-    </xacro:if>
   </xacro:macro>
 </robot>

File: robots/tmrv0_2/tmrv0_2.urdf.xacro (robot description, xacro)
@@ -5,12 +5,4 @@
   <!-- The ID of the robot model to be used -->
   <xacro:arg name="robot_type" default="tmrv0_2"/>
-  <!-- Is the robot being controlled with ros2_control?" -->
-  <xacro:arg name="ros2_control" default="false"/>
-  <!-- IP address or hostname of the robot" -->
-  <xacro:arg name="robot_ip" default="172.16.0.4"/>
-  <!-- Should a fake hardware be used? -->
-  <xacro:arg name="use_fake_hardware" default="false"/>
-  <!-- Should fake sensors be used? -->
-  <xacro:arg name="fake_sensor_commands" default="false"/>
   <!-- Should the reduced kinematic version (without caster wheels) be used? -->
   <xacro:arg name="reduced_version" default="false"/>
@@ -20,8 +12,4 @@
   <xacro:arg name="robot_namespace" default=""/>
   <xacro:tmrv0_2 mobile_robot_type="$(arg robot_type)"
-    robot_ip="$(arg robot_ip)"
-    ros2_control="$(arg ros2_control)"
-    use_fake_hardware="$(arg use_fake_hardware)"
-    fake_sensor_commands="$(arg fake_sensor_commands)"
     reduced_version="$(arg reduced_version)"
     robot_namespace="$(arg robot_namespace)"

File: robots/tmrv0_2/tmrv0_2.xacro (robot description, xacro)
@@ -3,11 +3,5 @@
   <xacro:macro name="tmrv0_2"
     params="mobile_robot_type
-                  robot_ip:=''
-                  ros2_control:=true
-                  use_fake_hardware:=false
-                  fake_sensor_commands:=false
                   reduced_version:=false
-                  is_async:=false
-                  thread_priority:=50
                   robot_namespace:=''
                   gazebo:=false">
@@ -138,17 +132,4 @@
       <origin xyz="-0.3275 -0.2175 0.19065" rpy="0 ${pi} ${pi*7/4}"/>
     </joint>
-    <xacro:if value="${ros2_control}">
-      <xacro:include filename="$(find franka_description)/robots/tmrv0_2/tmrv0_2.ros2_control.xacro"/>
-      <xacro:tmrv0_2_ros2_control
-        mobile_robot_type="${mobile_robot_type}"
-        robot_ip="${robot_ip}"
-        use_fake_hardware="${use_fake_hardware}"
-        fake_sensor_commands="${fake_sensor_commands}"
-        robot_namespace="${robot_namespace}"
-        gazebo="${gazebo}"
-        is_async="${is_async}"
-        thread_priority="${thread_priority}"
-      />
-    </xacro:if>
   </xacro:macro>
 </robot>
