Commit message: fix: tmr inertials updated

File: robots/tmrv0_2/argo_drive.xacro (robot description, xacro)
@@ -34,5 +34,5 @@
       <inertial>
         <origin xyz="-0.00019 ${offset_wheel_sign*0.04522} 0.02947" rpy="0 0 0"/>
-        <mass value="11.5"/>
+        <mass value="7.0"/>
         <inertia
           ixx="0.07060497424"
@@ -53,7 +53,7 @@
         <origin xyz="0 0 0" rpy="0 0 0"/>
         <mass value="2.0"/>
-        <inertia ixx="0.1" ixy="0.0" ixz="0.0"
-                 iyy="0.1" iyz="0.0"
-                 izz="0.1"/>
+        <inertia ixx="0.001" ixy="0.0" ixz="0.0"
+                 iyy="0.001" iyz="0.0"
+                 izz="0.001"/>
       </inertial>
     </link>

File: robots/tmrv0_2/caster_wheel.xacro (robot description, xacro)
@@ -25,5 +25,5 @@
       <inertial>
         <origin xyz="-0.02365 0.00005 -0.03651" rpy="0 0 0"/>
-        <mass value="0.7"/>
+        <mass value="0.3"/>
         <inertia
           ixx="0.00049538079"
@@ -43,5 +43,5 @@
       <inertial>
           <origin xyz="0 0 0" rpy="0 0 0"/>
-          <mass value="0.01"/>
+          <mass value="0.2"/>
           <inertia ixx="0.0001" ixy="0.0" ixz="0.0"
                    iyy="0.0001" iyz="0.0"
@@ -75,5 +75,5 @@
       <inertial>
         <origin xyz="0 0 0" rpy="0 0 0"/>
-        <mass value="0.001"/>
+        <mass value="0.2"/>
         <inertia ixx="0.0001" ixy="0.0" ixz="0.0"
                  iyy="0.0001" iyz="0.0"

File: robots/tmrv0_2/rocker_arm.xacro (robot description, xacro)
@@ -20,10 +20,10 @@
         <mass value="5.183973"/>
         <inertia
-          ixx="0.077004518565"
-          ixy="-0.000040505686"
-          ixz="-0.000026300402"
-          iyy="0.030693821144"
-          iyz="0.002939677599"
-          izz="0.083485865094"/>
+          ixx="0.067087560015"
+          ixy="-0.000078335851"
+          ixz="0.000041831678"
+          iyy="0.023113173265"
+          iyz="0.007148473123"
+          izz="0.081148329632"/>
       </inertial>
     </link>
