Commit message: refactor: Moved the origin of the fr3_duo_mount to 0 0 0 + moved kinematics/inertials out

File: accessories/fr3_duo_mount_v0_3/fr3_duo_mount.xacro (robot description, xacro)
@@ -4,8 +4,8 @@
   <xacro:property name="mount_kinematics"
     value="${xacro.load_yaml('$(find franka_description)/accessories/fr3_duo_mount_v0_3/kinematics.yaml')}"/>
-  <xacro:property name="inertials"
-    value="${xacro.load_yaml('$(find franka_description)/accessories/fr3_duo_mount_v0_3/inertials.yaml')}"/>
   <xacro:macro name="mount" params="name parent left_prefix right_prefix">
-    <link name="duo_mount_origin">
+    <xacro:property name="inertials"
+      value="${xacro.load_yaml('$(find franka_description)/accessories/fr3_duo_mount_v0_3/inertials.yaml')}"/>
+    <link name="fr3_duo_mount_mounting_point">
       <visual>
         <geometry>
@@ -36,35 +36,37 @@
       <xacro:franka-inertials name="mount"/>
     </link>
-    <link name="duo_mount_center"/>
-    <joint name="duo_mount_center_joint" type="fixed">
-      <parent link="duo_mount_origin"/>
-      <child link="duo_mount_center"/>
+    <link name="fr3_duo_mount_origin"/>
+    <joint name="fr3_duo_mount_origin_joint" type="fixed">
+      <parent link="fr3_duo_mount_mounting_point"/>
+      <child link="fr3_duo_mount_origin"/>
       <origin
-        xyz="${mount_kinematics['duo_mount_center']['kinematic']['x']} ${mount_kinematics['duo_mount_center']['kinematic']['y']} ${mount_kinematics['duo_mount_center']['kinematic']['z']}"
-        rpy="${mount_kinematics['duo_mount_center']['kinematic']['roll']} ${mount_kinematics['duo_mount_center']['kinematic']['pitch']} ${mount_kinematics['duo_mount_center']['kinematic']['yaw']}"/>
+        xyz="${-mount_kinematics['fr3_duo_mount_mounting_point']['kinematic']['x']} ${-mount_kinematics['fr3_duo_mount_mounting_point']['kinematic']['y']} ${-mount_kinematics['fr3_duo_mount_mounting_point']['kinematic']['z']}"
+        rpy="${-mount_kinematics['fr3_duo_mount_mounting_point']['kinematic']['roll']} ${-mount_kinematics['fr3_duo_mount_mounting_point']['kinematic']['pitch']} ${-mount_kinematics['fr3_duo_mount_mounting_point']['kinematic']['yaw']}"/>
     </joint>
     <!-- Mounting points for left and right robot -->
-    <link name="duo_mount_${left_prefix}"/>
-    <joint name="duo_mount_${left_prefix}_joint" type="fixed">
-      <parent link="duo_mount_center"/>
-      <child link="duo_mount_${left_prefix}"/>
+    <link name="fr3_duo_mount_${left_prefix}"/>
+    <joint name="fr3_duo_mount_${left_prefix}_joint" type="fixed">
+      <parent link="fr3_duo_mount_origin"/>
+      <child link="fr3_duo_mount_${left_prefix}"/>
       <origin
-        xyz="${mount_kinematics['duo_mount_left']['kinematic']['x']} ${mount_kinematics['duo_mount_left']['kinematic']['y']} ${mount_kinematics['duo_mount_left']['kinematic']['z']}"
-        rpy="${mount_kinematics['duo_mount_left']['kinematic']['roll']} ${mount_kinematics['duo_mount_left']['kinematic']['pitch']} ${mount_kinematics['duo_mount_left']['kinematic']['yaw']}"/>
+        xyz="${mount_kinematics['fr3_duo_mount_left']['kinematic']['x']} ${mount_kinematics['fr3_duo_mount_left']['kinematic']['y']} ${mount_kinematics['fr3_duo_mount_left']['kinematic']['z']}"
+        rpy="${mount_kinematics['fr3_duo_mount_left']['kinematic']['roll']} ${mount_kinematics['fr3_duo_mount_left']['kinematic']['pitch']} ${mount_kinematics['fr3_duo_mount_left']['kinematic']['yaw']}"/>
     </joint>
-    <link name="duo_mount_${right_prefix}">
+    <link name="fr3_duo_mount_${right_prefix}">
     </link>
-    <joint name="duo_mount_${right_prefix}_joint" type="fixed">
-      <parent link="duo_mount_center"/>
-      <child link="duo_mount_${right_prefix}"/>
+    <joint name="fr3_duo_mount_${right_prefix}_joint" type="fixed">
+      <parent link="fr3_duo_mount_origin"/>
+      <child link="fr3_duo_mount_${right_prefix}"/>
       <origin
-        xyz="${mount_kinematics['duo_mount_right']['kinematic']['x']} ${mount_kinematics['duo_mount_right']['kinematic']['y']} ${mount_kinematics['duo_mount_right']['kinematic']['z']}"
-        rpy="${mount_kinematics['duo_mount_right']['kinematic']['roll']} ${mount_kinematics['duo_mount_right']['kinematic']['pitch']} ${mount_kinematics['duo_mount_right']['kinematic']['yaw']}"/>
+        xyz="${mount_kinematics['fr3_duo_mount_right']['kinematic']['x']} ${mount_kinematics['fr3_duo_mount_right']['kinematic']['y']} ${mount_kinematics['fr3_duo_mount_right']['kinematic']['z']}"
+        rpy="${mount_kinematics['fr3_duo_mount_right']['kinematic']['roll']} ${mount_kinematics['fr3_duo_mount_right']['kinematic']['pitch']} ${mount_kinematics['fr3_duo_mount_right']['kinematic']['yaw']}"/>
     </joint>
-    <!-- The mount fixing the duo mount to the parent link -->
+    <!-- The mount fixing the duo mount to the parent link with the identity transform -->
     <joint name="mount_joint" type="fixed">
       <parent link="${parent}"/>
-      <child link="duo_mount_origin"/>
-      <origin xyz="0.0 0.0 0.0" rpy="0.0 0.0 0.0"/>
+      <child link="fr3_duo_mount_mounting_point"/>
+      <origin
+        xyz="0 0 0"
+        rpy="0 0 0"/>
     </joint>
   </xacro:macro>

File: accessories/franka_head_v0_2/franka_head.xacro (robot description, xacro)
@@ -1,5 +1,10 @@
 <?xml version="1.0" encoding="utf-8"?>
 <robot xmlns:xacro="http://www.ros.org/wiki/xacro">
+  <xacro:include filename="$(find franka_description)/robots/common/utils.xacro"/>
+  <xacro:property name="head_kinematics"
+    value="${xacro.load_yaml('$(find franka_description)/accessories/franka_head_v0_2/kinematics.yaml')}"/>
   <xacro:macro name="head" params="parent">
+    <xacro:property name="inertials"
+      value="${xacro.load_yaml('$(find franka_description)/accessories/franka_head_v0_2/inertials.yaml')}"/>
     <link name="head_link">
       <visual>
@@ -13,26 +18,22 @@
         </geometry>
       </collision>
-      <inertial>
-        <mass value="1.0"/>
-        <origin xyz="0 0 0" rpy="0 0 0"/>
-        <inertia ixx="0.01" ixy="0.0" ixz="0.0" iyy="0.01" iyz="0.0" izz="0.01"/>
-      </inertial>
+      <xacro:franka-inertials name="head"/>
     </link>
     <joint name="head_joint" type="fixed">
       <parent link="${parent}"/>
       <child link="head_link"/>
-      <origin xyz="0 0 0.167" rpy="0 0 0"/>
+      <origin
+        xyz="${head_kinematics['head']['kinematic']['x']} ${head_kinematics['head']['kinematic']['y']} ${head_kinematics['head']['kinematic']['z']}"
+        rpy="${head_kinematics['head']['kinematic']['roll']} ${head_kinematics['head']['kinematic']['pitch']} ${head_kinematics['head']['kinematic']['yaw']}"/>
     </joint>
     <link name="head_camera_mounting_point">
-      <inertial>
-        <mass value="0.001"/>
-        <origin xyz="0 0 0" rpy="0 0 0"/>
-        <inertia ixx="0.001" ixy="0.0" ixz="0.0" iyy="0.001" iyz="0.0" izz="0.001"/>
-      </inertial>
+      <xacro:franka-inertials name="head_camera_mounting_point"/>
     </link>
     <joint name="head_camera_mounting_point_joint" type="fixed">
-      <origin xyz="0.0498 -0.02 0.2345" rpy="0 0.7156 0"/>
       <parent link="head_link"/>
       <child link="head_camera_mounting_point"/>
+      <origin
+        xyz="${head_kinematics['head_camera_mounting_point']['kinematic']['x']} ${head_kinematics['head_camera_mounting_point']['kinematic']['y']} ${head_kinematics['head_camera_mounting_point']['kinematic']['z']}"
+        rpy="${head_kinematics['head_camera_mounting_point']['kinematic']['roll']} ${head_kinematics['head_camera_mounting_point']['kinematic']['pitch']} ${head_kinematics['head_camera_mounting_point']['kinematic']['yaw']}"/>
     </joint>
   </xacro:macro>

File: accessories/franka_spine_v0_1/franka_spine.xacro (robot description, xacro)
@@ -1,17 +1,20 @@
 <?xml version="1.0" encoding="utf-8"?>
 <robot xmlns:xacro="http://www.ros.org/wiki/xacro">
+  <xacro:include filename="$(find franka_description)/robots/common/utils.xacro"/>
+  <xacro:property name="spine_kinematics"
+    value="${xacro.load_yaml('$(find franka_description)/accessories/franka_spine_v0_1/kinematics.yaml')}"/>
   <!-- The spine is attached to 'parent' and provides a mounting point for other components -->
   <xacro:macro name="franka_spine" params="parent">
+    <xacro:property name="inertials"
+      value="${xacro.load_yaml('$(find franka_description)/accessories/franka_spine_v0_1/inertials.yaml')}"/>
     <joint name="franka_spine_fixed_joint" type="fixed">
       <parent link="${parent}"/>
       <child link="franka_spine"/>
-      <origin xyz="0.138289 0.0 0.350" rpy="0 0 0"/>
+      <origin
+        xyz="${spine_kinematics['franka_spine_fixed_joint']['kinematic']['x']} ${spine_kinematics['franka_spine_fixed_joint']['kinematic']['y']} ${spine_kinematics['franka_spine_fixed_joint']['kinematic']['z']}"
+        rpy="${spine_kinematics['franka_spine_fixed_joint']['kinematic']['roll']} ${spine_kinematics['franka_spine_fixed_joint']['kinematic']['pitch']} ${spine_kinematics['franka_spine_fixed_joint']['kinematic']['yaw']}"/>
     </joint>
     <link name="franka_spine_mounting_point">
-      <inertial>
-        <origin xyz="0 0 0" rpy="0 0 0"/>
-        <mass value="0.01"/>
-        <inertia ixx="0.0001" ixy="0.0" ixz="0.0" iyy="0.0001" iyz="0.0" izz="0.0001"/>
-      </inertial>
+      <xacro:franka-inertials name="franka_spine_mounting_point"/>
     </link>
     <link name="franka_spine">
@@ -29,15 +32,12 @@
         </material>
       </collision>
-      <inertial>
-        <origin xyz="0.042358 0.000378 0.495198" rpy="0 0 0"/>
-        <mass value="21.909124"/>
-        <inertia ixx="3.338968145" ixy="-0.000642887" ixz="0.299962762" iyy="3.324560297" iyz="-0.004488422"
-          izz="0.281489258"/>
-      </inertial>
+      <xacro:franka-inertials name="franka_spine"/>
     </link>
     <joint name="franka_spine_vertical_joint" type="prismatic">
       <parent link="franka_spine"/>
       <child link="franka_spine_mounting_point"/>
-      <origin xyz="0.266711 0.0 0.1" rpy="0 0 0"/>
+      <origin
+        xyz="${spine_kinematics['franka_spine_vertical_joint']['kinematic']['x']} ${spine_kinematics['franka_spine_vertical_joint']['kinematic']['y']} ${spine_kinematics['franka_spine_vertical_joint']['kinematic']['z']}"
+        rpy="${spine_kinematics['franka_spine_vertical_joint']['kinematic']['roll']} ${spine_kinematics['franka_spine_vertical_joint']['kinematic']['pitch']} ${spine_kinematics['franka_spine_vertical_joint']['kinematic']['yaw']}"/>
       <axis xyz="0 0 1"/>
       <limit effort="100" lower="0.0" upper="0.85" velocity="0.1"/>

File: robots/fr3_duo/fr3_duo.xacro (robot description, xacro)
@@ -45,5 +45,5 @@
         <!-- Attach the robot arm to the mount -->
         <joint name="${arm_prefixes_list[i]}_base_joint" type="fixed">
-          <parent link="duo_mount_${arm_prefixes_list[i]}"/>
+          <parent link="fr3_duo_mount_${arm_prefixes_list[i]}"/>
           <child link="${arm_prefixes_list[i]}_base"/>
         </joint>

File: robots/mobile_fr3_duo_v0_2/mobile_fr3_duo_v0_2.xacro (robot description, xacro)
@@ -61,5 +61,5 @@
     <!-- Head and Spine -->
     <xacro:franka_spine parent="base_link"/>
-    <xacro:head parent="duo_mount_origin"/>
+    <xacro:head parent="fr3_duo_mount_mounting_point"/>
     <!-- The FR3 Duo Arms -->
     <xacro:property name="only_arm_robot_types_list" value="${robot_types_list[1:]}"/>
